Commit message: new_simulation env

File: src/fire_description/urdf/fire_robot.xacro (robot description, xacro)
@@ -78,4 +78,32 @@
   </gazebo>
 <!--##############################################################-->
+<!--####################camera view############################-->
+  <link name="cam_follow_link">
+    <inertial>
+      <mass value="0.0001"/>
+      <inertia ixx="1e-6" ixy="0" ixz="0" iyy="1e-6" iyz="0" izz="1e-6"/>
+    </inertial>
+    <visual>
+      <geometry>
+        <sphere radius="0.1"/>
+      </geometry>
+      <material><color rgba="1 0 0 1"/></material>
+    </visual>
+    <collision>
+      <geometry>
+        <sphere radius="0.1"/>
+      </geometry>
+    </collision>
+  </link>
+  <!-- joint: fixed → revolute(잠금) -->
+  <joint name="cam_follow_joint" type="revolute">
+    <parent link="base_link"/>
+    <child link="cam_follow_link"/>
+    <origin xyz="0.05 0 0.3" rpy="0 0 3.1415926535"/>
+    <axis xyz="1 0 0"/>
+    <limit lower="0.0" upper="0.0" effort="0.1" velocity="0.1"/>
+    <dynamics damping="1.0"/>
+  </joint>
+<!--##############################################################-->
   <!-- ========== ARM ========== -->
   <joint name="arm_joint" type="revolute">
@@ -138,4 +166,5 @@
   <!--##############################################################-->
   <!-- ========== LEFT WHEELS (parent=base_link) ========== -->
+  <!-- ==================== left_wheel1 =================== -->
   <joint name="left_wheel_1_joint" type="continuous">
     <origin xyz="-0.2935 -0.15743 0" rpy="0 0 0"/>
@@ -163,4 +192,5 @@
   </gazebo>
 <!--##############################################################-->
+<!-- ==================== left_wheel2 =================== -->
   <joint name="left_wheel_2_joint" type="continuous">
     <origin xyz="0.025 -0.15743 0" rpy="0 0 0"/>
@@ -188,4 +218,5 @@
   </gazebo>
 <!--##############################################################-->
+<!-- ==================== left_wheel3 =================== -->
   <joint name="left_wheel_3_joint" type="continuous">
     <origin xyz="0.3455 -0.15743 0" rpy="0 0 0"/>
@@ -214,4 +245,5 @@
 <!--##############################################################-->
   <!-- ========== RIGHT WHEELS ========== -->
+  <!-- ========== right_wheel1 ========== -->
   <joint name="right_wheel_1_joint" type="continuous">
     <origin xyz="-0.2935 0.15743 0" rpy="0 0 0"/>
@@ -239,4 +271,5 @@
   </gazebo>
 <!--##############################################################-->
+<!-- ========== right_wheel2 ========== -->
   <joint name="right_wheel_2_joint" type="continuous">
     <origin xyz="0.025 0.15743 0" rpy="0 0 0"/>
@@ -264,4 +297,5 @@
   </gazebo>
 <!--##############################################################-->
+<!-- ========== right_wheel3 ========== -->
   <joint name="right_wheel_3_joint" type="continuous">
     <origin xyz="0.3455 0.15743 0" rpy="0 0 0"/>

Commit message: feat: sensors

File: src/fire_description/urdf/fire_robot.xacro (robot description, xacro)
@@ -1,14 +1,8 @@
 <?xml version="1.0"?>
 <robot xmlns:xacro="http://ros.org/wiki/xacro" name="fire_robot">
-<!--##############################################################-->
-<!--#################### XACRO 상수 ####################-->
+  <!-- XACRO constants -->
   <xacro:arg name="include_inertial" default="true"/>
-  <xacro:property name="mesh_dir"   value="$(find fire_description)/meshes"/>
-<!--##############################################################-->
-<!--#################### Robot Links & Joints ####################-->
-<!--##############################################################-->
-<!--##############################################################-->
-<!-- Base footprint link -->
-  <!-- xacro 루트 링크에 inertial 있으면 경고 띄움. dummy용-->
+  <xacro:property name="mesh_dir" value="$(find fire_description)/meshes"/>
+  <!-- Base footprint (dummy) -->
   <link name="base_footprint"/>
   <joint name="base_footprint_joint" type="fixed">
@@ -17,6 +11,5 @@
     <origin xyz="0 0 0.3" rpy="0 0 0"/>
   </joint>
-<!--##############################################################-->
-  <!-- ========== base_link (루트) ========== -->
+  <!-- base_link -->
   <link name="base_link">
     <inertial>
@@ -38,19 +31,21 @@
     </collision>
   </link>
-<!--##############################################################-->
-  <!-- ===== IMU frame ===== -->
+  <!-- IMU frame -->
   <link name="imu_link"/>
   <joint name="imu_joint" type="fixed">
     <parent link="base_link"/>
     <child link="imu_link"/>
-    <!-- 로봇 기준에서 IMU 위치/자세 조정 -->
     <origin xyz="-0.10 0.0 0.0" rpy="0 0 0"/>
   </joint>
-  <!-- ===== Gazebo Sim sensors on imu_link ===== -->
+  <!-- Gazebo Sim sensors (Fortress): use model-scoped topics to avoid collisions -->
   <gazebo reference="imu_link">
-    <!-- 6축 IMU(가속도+자이로) -->
+    <!-- IMU -->
     <sensor name="imu_sensor" type="imu">
-      <topic>/imu</topic>           <!-- GZ Transport topic -->
+      <topic>~/imu</topic>
       <update_rate>100</update_rate>
+      <plugin filename="libignition-gazebo-imu-system.so"
+                name="ignition::gazebo::systems::Imu"
+                />
+      <gz_frame_id>imu_link</gz_frame_id>
       <imu>
         <angular_velocity>
@@ -66,8 +61,12 @@
       </imu>
     </sensor>
-    <!-- 자력계(3축) -->
+    <!-- Magnetometer -->
     <sensor name="mag_sensor" type="magnetometer">
-      <topic>/mag</topic>           <!-- GZ Transport topic -->
+      <topic>~/mag</topic>
       <update_rate>50</update_rate>
+      <plugin filename="libignition-gazebo-magnetometer-system.so"
+                name="ignition::gazebo::systems::Magnetometer"
+                />
+      <gz_frame_id>imu_link</gz_frame_id>
       <magnetometer>
         <x><noise type="gaussian"><mean>0</mean><stddev>0.0005</stddev></noise></x>
@@ -77,6 +76,5 @@
     </sensor>
   </gazebo>
-<!--##############################################################-->
-<!--####################camera view############################-->
+  <!-- camera follow (helper) -->
   <link name="cam_follow_link">
     <inertial>
@@ -86,25 +84,24 @@
     <visual>
       <geometry>
-        <sphere radius="0.1"/>
-      </geometry>
-      <material><color rgba="1 0 0 1"/></material>
-    </visual>
-    <collision>
-      <geometry>
-        <sphere radius="0.1"/>
-      </geometry>
-    </collision>
-  </link>
-  <!-- joint: fixed → revolute(잠금) -->
+        <sphere radius="0.01"/>
+      </geometry>
+      <!-- URDF needs a material name attribute -->
+      <material name="cam_follow_red"><color rgba="1 0 0 1"/></material>
+    </visual>
+    <collision>
+      <geometry>
+        <sphere radius="0.001"/>
+      </geometry>
+    </collision>
+  </link>
   <joint name="cam_follow_joint" type="revolute">
     <parent link="base_link"/>
     <child link="cam_follow_link"/>
-    <origin xyz="0.05 0 0.3" rpy="0 0 3.1415926535"/>
+    <origin xyz="0.05 0 0.5" rpy="0 0 3.1415926535"/>
     <axis xyz="1 0 0"/>
     <limit lower="0.0" upper="0.0" effort="0.1" velocity="0.1"/>
     <dynamics damping="1.0"/>
   </joint>
-<!--##############################################################-->
-  <!-- ========== ARM ========== -->
+  <!-- ARM -->
   <joint name="arm_joint" type="revolute">
     <origin xyz="0.2765 0 0" rpy="0 0 0"/>
@@ -112,6 +109,5 @@
     <child link="arm"/>
     <axis xyz="0 1 0"/>
-    <limit velocity="1.0" lower="-0.5" upper="0.5" effort="50" />
-    <!-- dynamic damping -->
+    <limit velocity="1.0" lower="-0.5" upper="0.5" effort="50"/>
     <dynamics damping="0.05" friction="0.2"/>
   </joint>
@@ -135,6 +131,5 @@
     </collision>
   </link>
-<!--##############################################################-->
-  <!-- ========== BLADE ========== -->
+  <!-- BLADE -->
   <joint name="blade_joint" type="continuous">
     <origin xyz="0.240 0 0" rpy="0 0 0"/>
@@ -164,7 +159,5 @@
     </collision>
   </link>
-  <!--##############################################################-->
-  <!-- ========== LEFT WHEELS (parent=base_link) ========== -->
-  <!-- ==================== left_wheel1 =================== -->
+  <!-- LEFT WHEELS -->
   <joint name="left_wheel_1_joint" type="continuous">
     <origin xyz="-0.2935 -0.15743 0" rpy="0 0 0"/>
@@ -175,22 +168,14 @@
   <link name="left_wheel1">
     <inertial><origin xyz="0 0 0" rpy="0 0 0"/>
-      <mass value="2.5"/><inertia ixx="0.002" ixy="0" ixz="0" iyy="0.002" iyz="0" izz="0.002"/></inertial>
-    <visual>
-      <origin xyz="0 0 0" rpy="0 0 0"/>
-      <geometry><mesh filename="file://${mesh_dir}/left_wheel.obj" scale="0.01 0.01 0.01"/></geometry>
-    </visual>
-    <collision>
-      <origin xyz="0 0 0" rpy="0 0 0"/>
-      <geometry><mesh filename="file://${mesh_dir}/left_wheel.obj" scale="0.01 0.01 0.01"/></geometry>
-    </collision>
-  </link>
-  <gazebo reference="left_wheel1">
-    <mu1>1.0</mu1>   <!-- 표면 마찰 계수 -->
-    <mu2>1.0</mu2>
-    <kp>1e5</kp>     <!-- 접촉 강성 -->
-    <kd>1.0</kd>     <!-- 접촉 감쇠 -->
-  </gazebo>
-<!--##############################################################-->
-<!-- ==================== left_wheel2 =================== -->
+      <mass value="2.5"/><inertia ixx="0.0068" ixy="0" ixz="0" iyy="0.0068" iyz="0" izz="0.0125"/></inertial>
+    <visual>
+      <origin xyz="0 0 0" rpy="0 0 0"/>
+      <geometry><mesh filename="file://${mesh_dir}/left_wheel.obj" scale="0.01 0.01 0.01"/></geometry>
+    </visual>
+    <collision>
+      <origin xyz="0 0 0" rpy="0 0 0"/>
+      <geometry><mesh filename="file://${mesh_dir}/left_wheel.obj" scale="0.01 0.01 0.01"/></geometry>
+    </collision>
+  </link>
   <joint name="left_wheel_2_joint" type="continuous">
     <origin xyz="0.025 -0.15743 0" rpy="0 0 0"/>
@@ -201,22 +186,14 @@
   <link name="left_wheel2">
     <inertial><origin xyz="0 0 0" rpy="0 0 0"/>
-      <mass value="2.5"/><inertia ixx="0.002" ixy="0" ixz="0" iyy="0.002" iyz="0" izz="0.002"/></inertial>
-    <visual>
-      <origin xyz="0 0 0" rpy="0 0 0"/>
-      <geometry><mesh filename="file://${mesh_dir}/left_wheel.obj" scale="0.01 0.01 0.01"/></geometry>
-    </visual>
-    <collision>
-      <origin xyz="0 0 0" rpy="0 0 0"/>
-      <geometry><mesh filename="file://${mesh_dir}/left_wheel.obj" scale="0.01 0.01 0.01"/></geometry>
-    </collision>
-  </link>
-  <gazebo reference="left_wheel2">
-    <mu1>1.0</mu1>   <!-- 표면 마찰 계수 -->
-    <mu2>1.0</mu2>
-    <kp>1e5</kp>     <!-- 접촉 강성 -->
-    <kd>1.0</kd>     <!-- 접촉 감쇠 -->
-  </gazebo>
-<!--##############################################################-->
-<!-- ==================== left_wheel3 =================== -->
+      <mass value="2.5"/><inertia ixx="0.0068" ixy="0" ixz="0" iyy="0.0068" iyz="0" izz="0.0125"/></inertial>
+    <visual>
+      <origin xyz="0 0 0" rpy="0 0 0"/>
+      <geometry><mesh filename="file://${mesh_dir}/left_wheel.obj" scale="0.01 0.01 0.01"/></geometry>
+    </visual>
+    <collision>
+      <origin xyz="0 0 0" rpy="0 0 0"/>
+      <geometry><mesh filename="file://${mesh_dir}/left_wheel.obj" scale="0.01 0.01 0.01"/></geometry>
+    </collision>
+  </link>
   <joint name="left_wheel_3_joint" type="continuous">
     <origin xyz="0.3455 -0.15743 0" rpy="0 0 0"/>
@@ -227,23 +204,15 @@
   <link name="left_wheel3">
     <inertial><origin xyz="0 0 0" rpy="0 0 0"/>
-      <mass value="2.5"/><inertia ixx="0.002" ixy="0" ixz="0" iyy="0.002" iyz="0" izz="0.002"/></inertial>
-    <visual>
-      <origin xyz="0 0 0" rpy="0 0 0"/>
-      <geometry><mesh filename="file://${mesh_dir}/left_wheel.obj" scale="0.01 0.01 0.01"/></geometry>
-    </visual>
-    <collision>
-      <origin xyz="0 0 0" rpy="0 0 0"/>
-      <geometry><mesh filename="file://${mesh_dir}/left_wheel.obj" scale="0.01 0.01 0.01"/></geometry>
-    </collision>
-  </link>
-  <gazebo reference="left_wheel3">
-    <mu1>1.0</mu1>   <!-- 표면 마찰 계수 -->
-    <mu2>1.0</mu2>
-    <kp>1e5</kp>     <!-- 접촉 강성 -->
-    <kd>1.0</kd>     <!-- 접촉 감쇠 -->
-  </gazebo>
-<!--##############################################################-->
-  <!-- ========== RIGHT WHEELS ========== -->
-  <!-- ========== right_wheel1 ========== -->
+      <mass value="2.5"/><inertia ixx="0.0068" ixy="0" ixz="0" iyy="0.0068" iyz="0" izz="0.0125"/></inertial>
+    <visual>
+      <origin xyz="0 0 0" rpy="0 0 0"/>
+      <geometry><mesh filename="file://${mesh_dir}/left_wheel.obj" scale="0.01 0.01 0.01"/></geometry>
+    </visual>
+    <collision>
+      <origin xyz="0 0 0" rpy="0 0 0"/>
+      <geometry><mesh filename="file://${mesh_dir}/left_wheel.obj" scale="0.01 0.01 0.01"/></geometry>
+    </collision>
+  </link>
+  <!-- RIGHT WHEELS -->
   <joint name="right_wheel_1_joint" type="continuous">
     <origin xyz="-0.2935 0.15743 0" rpy="0 0 0"/>
@@ -254,22 +223,14 @@
   <link name="right_wheel1">
     <inertial><origin xyz="0 0 0" rpy="0 0 0"/>
-      <mass value="2.5"/><inertia ixx="0.002" ixy="0" ixz="0" iyy="0.002" iyz="0" izz="0.002"/></inertial>
-    <visual>
-      <origin xyz="0 0 0" rpy="0 0 0"/>
-      <geometry><mesh filename="file://${mesh_dir}/right_wheel.obj" scale="0.01 0.01 0.01"/></geometry>
-    </visual>
-    <collision>
-      <origin xyz="0 0 0" rpy="0 0 0"/>
-      <geometry><mesh filename="file://${mesh_dir}/right_wheel.obj" scale="0.01 0.01 0.01"/></geometry>
-    </collision>
-  </link>
-  <gazebo reference="right_wheel1">
-    <mu1>1.0</mu1>   <!-- 표면 마찰 계수 -->
-    <mu2>1.0</mu2>
-    <kp>1e5</kp>     <!-- 접촉 강성 -->
-    <kd>1.0</kd>     <!-- 접촉 감쇠 -->
-  </gazebo>
-<!--##############################################################-->
-<!-- ========== right_wheel2 ========== -->
+      <mass value="2.5"/><inertia ixx="0.0068" ixy="0" ixz="0" iyy="0.0068" iyz="0" izz="0.0125"/></inertial>
+    <visual>
+      <origin xyz="0 0 0" rpy="0 0 0"/>
+      <geometry><mesh filename="file://${mesh_dir}/right_wheel.obj" scale="0.01 0.01 0.01"/></geometry>
+    </visual>
+    <collision>
+      <origin xyz="0 0 0" rpy="0 0 0"/>
+      <geometry><mesh filename="file://${mesh_dir}/right_wheel.obj" scale="0.01 0.01 0.01"/></geometry>
+    </collision>
+  </link>
   <joint name="right_wheel_2_joint" type="continuous">
     <origin xyz="0.025 0.15743 0" rpy="0 0 0"/>
@@ -280,22 +241,14 @@
   <link name="right_wheel2">
     <inertial><origin xyz="0 0 0" rpy="0 0 0"/>
-      <mass value="2.5"/><inertia ixx="0.002" ixy="0" ixz="0" iyy="0.002" iyz="0" izz="0.002"/></inertial>
-    <visual>
-      <origin xyz="0 0 0" rpy="0 0 0"/>
-      <geometry><mesh filename="file://${mesh_dir}/right_wheel.obj" scale="0.01 0.01 0.01"/></geometry>
-    </visual>
-    <collision>
-      <origin xyz="0 0 0" rpy="0 0 0"/>
-      <geometry><mesh filename="file://${mesh_dir}/right_wheel.obj" scale="0.01 0.01 0.01"/></geometry>
-    </collision>
-  </link>
-  <gazebo reference="right_wheel2">
-    <mu1>1.0</mu1>   <!-- 표면 마찰 계수 -->
-    <mu2>1.0</mu2>
-    <kp>1e5</kp>     <!-- 접촉 강성 -->
-    <kd>1.0</kd>     <!-- 접촉 감쇠 -->
-  </gazebo>
-<!--##############################################################-->
-<!-- ========== right_wheel3 ========== -->
+      <mass value="2.5"/><inertia ixx="0.0068" ixy="0" ixz="0" iyy="0.0068" iyz="0" izz="0.0125"/></inertial>
+    <visual>
+      <origin xyz="0 0 0" rpy="0 0 0"/>
+      <geometry><mesh filename="file://${mesh_dir}/right_wheel.obj" scale="0.01 0.01 0.01"/></geometry>
+    </visual>
+    <collision>
+      <origin xyz="0 0 0" rpy="0 0 0"/>
+      <geometry><mesh filename="file://${mesh_dir}/right_wheel.obj" scale="0.01 0.01 0.01"/></geometry>
+    </collision>
+  </link>
   <joint name="right_wheel_3_joint" type="continuous">
     <origin xyz="0.3455 0.15743 0" rpy="0 0 0"/>
@@ -306,26 +259,19 @@
   <link name="right_wheel3">
     <inertial><origin xyz="0 0 0" rpy="0 0 0"/>
-      <mass value="2.5"/><inertia ixx="0.002" ixy="0" ixz="0" iyy="0.002" iyz="0" izz="0.002"/></inertial>
-    <visual>
-      <origin xyz="0 0 0" rpy="0 0 0"/>
-      <geometry><mesh filename="file://${mesh_dir}/right_wheel.obj" scale="0.01 0.01 0.01"/></geometry>
-    </visual>
-    <collision>
-      <origin xyz="0 0 0" rpy="0 0 0"/>
-      <geometry><mesh filename="file://${mesh_dir}/right_wheel.obj" scale="0.01 0.01 0.01"/></geometry>
-    </collision>
-  </link>
-  <gazebo reference="right_wheel3">
-    <mu1>1.0</mu1>   <!-- 표면 마찰 계수 -->
-    <mu2>1.0</mu2>
-    <kp>1e5</kp>     <!-- 접촉 강성 -->
-    <kd>1.0</kd>     <!-- 접촉 감쇠 -->
-  </gazebo>
-  <!-- ===== ros2_control: Gazebo Sim 하드웨어 플러그인 ===== -->
+      <mass value="2.5"/><inertia ixx="0.0068" ixy="0" ixz="0" iyy="0.0068" iyz="0" izz="0.0125"/></inertial>
+    <visual>
+      <origin xyz="0 0 0" rpy="0 0 0"/>
+      <geometry><mesh filename="file://${mesh_dir}/right_wheel.obj" scale="0.01 0.01 0.01"/></geometry>
+    </visual>
+    <collision>
+      <origin xyz="0 0 0" rpy="0 0 0"/>
+      <geometry><mesh filename="file://${mesh_dir}/right_wheel.obj" scale="0.01 0.01 0.01"/></geometry>
+    </collision>
+  </link>
+  <!-- ros2_control (Gazebo Sim) -->
   <ros2_control name="RobotController" type="system">
     <hardware>
       <plugin>gz_ros2_control/GazeboSimSystem</plugin>
     </hardware>
-    <!-- Arm : position 명령-->
     <joint name="arm_joint">
       <command_interface name="position"/>
@@ -335,5 +281,4 @@
       <state_interface name="effort"/>
     </joint>
-    <!-- Blade : velocity 명령-->
     <joint name="blade_joint">
       <command_interface name="velocity"/>
@@ -342,5 +287,9 @@
       <state_interface name="effort"/>
     </joint>
-    <!-- Wheels : velocity 명령-->
+    <!-- cam_follow_joint 추가 -->
+    <joint name="cam_follow_joint">
+      <state_interface name="position"/>
+      <state_interface name="velocity"/>
+    </joint>
     <joint name="left_wheel_1_joint"><command_interface name="velocity"/>
       <state_interface name="position"/><state_interface name="velocity"/></joint>
@@ -356,14 +305,8 @@
       <state_interface name="position"/><state_interface name="velocity"/></joint>
   </ros2_control>
-  <!-- ===== Gazebo 플러그인: 컨트롤러 매니저 구동 ===== -->
+  <!-- ros2_control plugin (Gazebo Sim) -->
   <gazebo>
-    <plugin filename="libgz_ros2_control-system.so"
-            name="gz_ros2_control::GazeboSimROS2ControlPlugin">
+    <plugin filename="libgz_ros2_control-system.so" name="gz_ros2_control::GazeboSimROS2ControlPlugin">
       <parameters>$(find fire_bringup)/config/controller.yaml</parameters>
-      <!-- 필요 시 네임스페이스/리매핑도 추가 가능
-      <ros>
-        <namespace>fire</namespace>
-      </ros>
-      -->
     </plugin>
   </gazebo>
